File: Shutter.sch (EAGLE design)
At the start: 44 parts, among them IC1 7805TV, IC2 7812TV, IC3 MAX3222, IC4 74AC00D, IC5 7808T, J1 ATMEL_PROGRAMMER_HEADERTH

Commit message: Updates to schematic. Definitely not done yet!
Parts:
- removed IC1: 7805TV, linear:7805TV
- added C18: 1u, ERIC:CAP5MM
- added C19: 100n, KEMET:CAP805B
- added J2: (no value), SparkFun-Connectors:M06NO_SILK_FEMALE_PTH
- added U$7: DPDTA_DP, NKK:DPDTA_DP
- added U1: (no value), ERIC:VOLTAGE_REGULATOR_LDOMCP1702_TO-92
- C1, C16, C2, C3, C4: value (none) -> 1u; device ERIC:CAP_POL5MMD_5MML -> ERIC:CAP5MM
- C17: value (none) -> 10u; device ERIC:CAP_POL5MMD_5MML -> ERIC:CAP_POL8_3.5
- renumbered IC2 to MC7812, IC5 to MC7808
Connections:
- net !Q! renamed SHUTTER_OPEN_LATCH
- net CS2 renamed SHUTTER_STATUS_PIN
- net N$10 renamed TX
- net N$11 renamed RX
- net RESET renamed RESET_CLOSE_SHUTTER
- net SET renamed SET_OPEN_SHUTTER
- removed net CS1: U$1.PD3(INT1)
- removed net EN1: D1G$5.!G!, U$1.PD5(T1), U$5.!RE!
- removed net EN2: D2G$5.!G!, U$1.PD6(AIN0), U$6.!RE!
- removed net N$26: D1G$4.Y
- removed net N$27: D1G$4.Z
- removed net N$28: D2G$4.Z
- removed net N$29: D2G$4.Y
- removed net Q: IC4A.O, IC4B.I0
- removed net RESET_PIN: U$1.PB1(OC1A)
- removed net SET_PIN: U$1.PB0(ICP)
- new net CLOSE_PIN: U$1.PD5(T1)
- new net DTR: C19.2, J2.6
- new net ENABLE1: D1G$5.!G!, U$1.PB1(OC1A), U$5.!RE!
- new net ENABLE2: D2G$5.!G!, U$1.PB0(ICP), U$6.!RE!
- new net FTDI_RX: J2.5, U$7.U1
- new net FTDI_TX: J2.4, U$7.U
- new net MAX_RX: IC3G$1.R1OUT, U$7.D1
- new net MAX_TX: IC3G$1.T1IN, U$7.D
- new net N$11: D2G$2.A
- new net OPEN_PIN: U$1.PD6(AIN0)
- new net SHUTTER_CLOSED_LATCH: IC4A.O, IC4B.I0, U$1.PD3(INT1)
- net 12V: now also C1.1, C2.1; no longer C16.+, C2.+
- net 24V: now also C17.+, C18.1; no longer C1.+
- net 5V: now also C16.1, U1.VOUT; no longer C4.+, IC1.VO
- net 8V: now also C3.1, C4.1, U1.VIN; no longer C17.+, C3.+, IC1.VI
- net CS: now also D1G$3.A, D2G$3.A; no longer D1G$1.A, D2G$1.A
- net CS+1: now also D1G$3.Y; no longer D1G$1.Y
- net CS+2: now also D2G$3.Y; no longer D2G$1.Y
- net CS-1: now also D1G$3.Z; no longer D1G$1.Z
- net CS-2: now also D2G$3.Z; no longer D2G$1.Z
- net GND: now also C1.2, C16.2, C18.2, C2.2, C3.2, C4.2, D1G$2.A, J2.1, U1.GND; no longer C1.-, C16.-, C2.-, C3.-, C4.-, D1G$4.A, D2G$4.A, IC1.GND
- net MOSI: now also D1G$4.A, D2G$4.A; no longer D1G$3.A, D2G$3.A
- net MOSI+1: now also D1G$4.Y; no longer D1G$3.Y
- net MOSI+2: now also D2G$4.Y; no longer D2G$3.Y
- net MOSI-1: now also D1G$4.Z; no longer D1G$3.Z
- net MOSI-2: now also D2G$4.Z; no longer D2G$3.Z
- net RST: now also C19.1
- net RXD: now also U$7.C1; no longer IC3G$1.R1OUT
- net SCK: now also D1G$1.A, D2G$1.A; no longer D1G$2.A, D2G$2.A
- net SCK+1: now also D1G$1.Y; no longer D1G$2.Y
- net SCK+2: now also D2G$1.Y; no longer D2G$2.Y
- net SCK-1: now also D1G$1.Z; no longer D1G$2.Z
- net SCK-2: now also D2G$1.Z; no longer D2G$2.Z
- net TXD: now also U$7.C; no longer IC3G$1.T1IN
Other:
- note added: "6 pin In Circuit Programmer Header for Atmel MkII"
- note added: "8V is distributed to ADC board"
- note added: "CTS not connected"
- note added: "Comm Switch"
- note added: "Connects to board ADC1"
- note added: "Connects to board ADC2"
- note added: "Currently unused"
- note added: "FTDI connector interface"
- note added: "MCP1702-500"
- note added: "NC"
- note added: "Overlap between this two pins?"
- note added: "Power for ADC 1 and fault signal"
- note added: "Power for ADC 2 and fault signal"
- note added: "Power not connected"
- note added: "Power's logic on board"
- note added: "Regulated Voltage Sources"
- note added: "Shutter not powered Shutter in closed position"
- note added: "Shutter powered Shutter in open position"
- note added: "Switches between the MAX3222 And FTDI interfaces"
- note added: "TO-220 package with heatsink"
- note added: "The MAX3222 is used to communicate via RS232. FTDI is used to comm with Arduino Software."
- note added: "Unused"
- note added: "Use 16MHz for Arduino compatibility"
- note added: "Yellow"
- note added: "brown"
- note added: "brown wire"
- note added: "characteristic impedance of cable"
- note added: "green"
- note added: "green wire"
- note added: "momentary push button"
- note added: "orange"
- note added: "orange wire"
- note added: "routed through comm switch"
- note added: "to pin 2 (RX) of DB9 Male"
- note added: "to pin 3 (TX) of DB9 Male"
- note added: "to pin 5 (GND) of DB9 Male"
- note added: "unused"
- note removed: "CAP values TBD"
- note removed: "Goes to MAX3222"
- note removed: "Q bar means shutter is open"
- note removed: "Q means shutter is down"
- note removed: "REGULATORS"
- note removed: "TO-92 package 1%"
- note removed: "Use a 7808 instead"
- note removed: "tO-220 package"
- moved on the sheet: ADC1_FAULT, ADC2_FAULT, C17, C5, C6, CO[, IC4P, U$4

Commit message: Update schematic to reflect current circuit. Change names of some nets to match sofware variables.
Parts:
- added D3: 1N4004, adafruit:1N4004
- added POWER, SHUTTER, SHUTTER_CLOSED_INDICATOR, SHUTTER_OPEN_INDICATOR: M02, OST:M02
- added R8: 1.6K, Stackpole:RESISTOR0805
- added T1: TIP131, transistor:TIP131
Connections:
- net CS renamed SS
- net N$16 renamed SHUTTER_FAULT
- removed net N$1: ADC1_FAULT.3
- removed net SHUTTER_STATUS_PIN: U$1.PD4(XCK/T0)
- new net DEWAR_DIFF_ENABLE: U$1.PD6(AIN0), U$5.!RE!
- new net DEWAR_FAULT: ADC1_FAULT.3, U$1.PD3(INT1)
- new net N$10: D3.A, SHUTTER.2, T1.C
- new net N$16: R8.1, T1.B
- new net SHUTTER_DIFF_ENABLE: U$1.PD5(T1), U$6.!RE!
- net 24V: now also D3.C, SHUTTER.1
- net 5V: now also POWER.1
- net CLOSE_PIN: now also U$1.PB0(ICP); no longer U$1.PD5(T1)
- net ENABLE1: no longer U$1.PB1(OC1A), U$5.!RE!
- net ENABLE2: no longer U$1.PB0(ICP), U$6.!RE!
- net GND: now also POWER.2, SHUTTER_CLOSED_INDICATOR.2, SHUTTER_OPEN_INDICATOR.2, T1.E
- net OPEN_PIN: now also U$1.PD7(AIN1); no longer U$1.PD6(AIN0)
- net SHUTTER_CLOSED_LATCH: now also SHUTTER_CLOSED_INDICATOR.1, U$1.PD2(INT0); no longer U$1.PD3(INT1)
- net SHUTTER_OPEN_LATCH: now also R8.2, SHUTTER_OPEN_INDICATOR.1
Other:
- note added: "BIGGER, with heat sink?"
- note added: "DEWAR DIFF DRIVERS"
- note added: "LED INDICATORS"
- note added: "TRIGGER"
- note added: "Used a TIP102 on board"
- note added: "reevaluate size of resistor"
- note removed: "First SPI connection"
- note removed: "NC"

Commit message: Added screw terminals for toggles.
Parts:
- added DEWAR_SWITCH, SHUTTER_SWITCH: M02, OST:M02
- added OPEN_CLOSE_TOGGLE: M03, OST:M03
Connections:
- new net DEWAR_FAULT_TRIGGER: DEWAR_SWITCH.2
- new net SHUTTER_FAULT_TRIGGER: SHUTTER_SWITCH.2
- net DEWAR_FAULT: now also DEWAR_SWITCH.1
- net GND: now also OPEN_CLOSE_TOGGLE.2
- net RESET_CLOSE_SHUTTER: now also OPEN_CLOSE_TOGGLE.1
- net SET_OPEN_SHUTTER: now also OPEN_CLOSE_TOGGLE.3
- net SHUTTER_FAULT: now also SHUTTER_SWITCH.1
Other:
- note added: "Connect to SPDT(MOM)(MOM) Switch"
- note added: "Reflex Circuit. Connect to 2PST"
- moved on the sheet: ADC1_FAULT, ADC2_FAULT
Changed lines of the file:
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@@
 <part name="R8" library="Stackpole" deviceset="RESISTOR" device="0805" value="1.6K"/>
 <part name="D3" library="adafruit" library_urn="urn:adsk.eagle:library:420" deviceset="1N4004" device=""/>
+<part name="DEWAR_SWITCH" library="OST" deviceset="M02" device=""/>
+<part name="SHUTTER_SWITCH" library="OST" deviceset="M02" device=""/>
+<part name="OPEN_CLOSE_TOGGLE" library="OST" deviceset="M03" device=""/>
+<part name="GND51" library="supply1" library_urn="urn:adsk.eagle:library:371" deviceset="GND" device=""/>
 </parts>
 <sheets>
@@
 <text x="276.86" y="66.04" size="2.54" layer="94">reevaluate size of resistor</text>
 <text x="335.28" y="78.74" size="1.778" layer="94">Used a TIP102 on board</text>
+<text x="-106.68" y="142.24" size="1.778" layer="94">Reflex Circuit.
+Connect to 2PST</text>
+<text x="-106.68" y="109.22" size="1.778" layer="94">Connect to SPDT(MOM)(MOM)
+Switch</text>
 </plain>
 <moduleinsts>
@@
 <instance part="ADC2" gate="G$1" x="325.12" y="167.64" rot="R180"/>
 <instance part="ADC1" gate="G$1" x="193.04" y="165.1" rot="R180"/>
-<instance part="ADC1_FAULT" gate="G$1" x="-25.4" y="132.08"/>
-<instance part="ADC2_FAULT" gate="G$1" x="-25.4" y="116.84"/>
-<instance part="GND43" gate="1" x="-15.24" y="116.84" rot="R90"/>
-<instance part="GND44" gate="1" x="-15.24" y="132.08" rot="R90"/>
+<instance part="ADC1_FAULT" gate="G$1" x="-33.02" y="137.16"/>
+<instance part="ADC2_FAULT" gate="G$1" x="-33.02" y="124.46"/>
+<instance part="GND43" gate="1" x="-17.78" y="124.46" rot="R90"/>
+<instance part="GND44" gate="1" x="-17.78" y="137.16" rot="R90"/>
 <instance part="V1" gate="G$1" x="-73.66" y="165.1"/>
 <instance part="GND37" gate="1" x="-58.42" y="160.02"/>
@@
 <instance part="R8" gate="G$1" x="312.42" y="81.28" rot="R180"/>
 <instance part="D3" gate="1" x="332.74" y="88.9" rot="R90"/>
+<instance part="DEWAR_SWITCH" gate="G$1" x="-99.06" y="134.62"/>
+<instance part="SHUTTER_SWITCH" gate="G$1" x="-99.06" y="121.92"/>
+<instance part="OPEN_CLOSE_TOGGLE" gate="G$1" x="-99.06" y="101.6"/>
+<instance part="GND51" gate="1" x="-81.28" y="101.6" rot="R90"/>
 </instances>
 <busses>
@@
 <pinref part="ADC2_FAULT" gate="G$1" pin="2"/>
 <pinref part="GND43" gate="1" pin="GND"/>
-</segment>
-<segment>
-<pinref part="ADC1_FAULT" gate="G$1" pin="2"/>
-<pinref part="GND44" gate="1" pin="GND"/>
+<wire x1="-25.4" y1="124.46" x2="-20.32" y2="124.46" width="0.1524" layer="91"/>
 </segment>
 <segment>
@@
 <pinref part="T1" gate="G$1" pin="E"/>
 <pinref part="GND50" gate="1" pin="GND"/>
+</segment>
+<segment>
+<pinref part="ADC1_FAULT" gate="G$1" pin="2"/>
+<pinref part="GND44" gate="1" pin="GND"/>
+<wire x1="-25.4" y1="137.16" x2="-20.32" y2="137.16" width="0.1524" layer="91"/>
+</segment>
+<segment>
+<pinref part="OPEN_CLOSE_TOGGLE" gate="G$1" pin="2"/>
+<pinref part="GND51" gate="1" pin="GND"/>
+<wire x1="-83.82" y1="101.6" x2="-91.44" y2="101.6" width="0.1524" layer="91"/>
 </segment>
 </net>
@@
 <label x="43.18" y="101.6" size="1.27" layer="95" font="vector" xref="yes"/>
 </segment>
+<segment>
+<pinref part="OPEN_CLOSE_TOGGLE" gate="G$1" pin="3"/>
+<wire x1="-91.44" y1="99.06" x2="-88.9" y2="99.06" width="0.1524" layer="91"/>
+<label x="-88.9" y="99.06" size="1.27" layer="95" xref="yes"/>
+</segment>
 </net>
 <net name="MISO+1" class="0">
@@
 <net name="DEWAR_FAULT" class="0">
 <segment>
-<pinref part="ADC1_FAULT" gate="G$1" pin="3"/>
-<portref moduleinst="BUFFER_OD1" port="A1"/>
-<wire x1="-17.78" y1="129.54" x2="0" y2="116.84" width="0.1524" layer="91"/>
-<label x="-12.7" y="127" size="1.27" layer="95" xref="yes"/>
-</segment>
-<segment>
 <pinref part="U$1" gate="G$1" pin="PD3(INT1)"/>
 <wire x1="116.84" y1="40.64" x2="119.38" y2="40.64" width="0.1524" layer="91"/>
 <label x="121.92" y="40.64" size="1.27" layer="95" xref="yes"/>
 </segment>
+<segment>
+<pinref part="DEWAR_SWITCH" gate="G$1" pin="1"/>
+<wire x1="-91.44" y1="137.16" x2="-88.9" y2="137.16" width="0.1524" layer="91"/>
+<label x="-88.9" y="137.16" size="1.27" layer="95" xref="yes"/>
+</segment>
+<segment>
+<pinref part="ADC1_FAULT" gate="G$1" pin="3"/>
+<wire x1="-25.4" y1="134.62" x2="-22.86" y2="134.62" width="0.1524" layer="91"/>
+<label x="-22.86" y="134.62" size="1.27" layer="95" xref="yes"/>
+</segment>
 </net>
 <net name="SHUTTER_FAULT" class="0">
 <segment>
+<pinref part="SHUTTER_SWITCH" gate="G$1" pin="1"/>
+<wire x1="-91.44" y1="124.46" x2="-88.9" y2="124.46" width="0.1524" layer="91"/>
+<label x="-88.9" y="124.46" size="1.27" layer="95" xref="yes"/>
+</segment>
+<segment>
 <pinref part="ADC2_FAULT" gate="G$1" pin="3"/>
-<portref moduleinst="BUFFER_OD1" port="A2"/>
-<wire x1="-17.78" y1="114.3" x2="0" y2="111.76" width="0.1524" layer="91"/>
-<label x="-10.16" y="114.3" size="1.27" layer="95" xref="yes"/>
+<wire x1="-25.4" y1="121.92" x2="-20.32" y2="121.92" width="0.1524" layer="91"/>
+<label x="-20.32" y="121.92" size="1.27" layer="95" xref="yes"/>
 </segment>
 </net>
@@
 <segment>
 <pinref part="ADC1_FAULT" gate="G$1" pin="1"/>
-<wire x1="-17.78" y1="134.62" x2="-15.24" y2="134.62" width="0.1524" layer="91"/>
-<label x="-15.24" y="134.62" size="1.27" layer="95" font="vector" xref="yes"/>
+<wire x1="-25.4" y1="139.7" x2="-22.86" y2="139.7" width="0.1524" layer="91"/>
+<label x="-22.86" y="139.7" size="1.27" layer="95" font="vector" xref="yes"/>
 </segment>
 <segment>
 <pinref part="ADC2_FAULT" gate="G$1" pin="1"/>
-<wire x1="-17.78" y1="119.38" x2="-15.24" y2="119.38" width="0.1524" layer="91"/>
-<label x="-15.24" y="119.38" size="1.27" layer="95" font="vector" xref="yes"/>
+<wire x1="-25.4" y1="127" x2="-22.86" y2="127" width="0.1524" layer="91"/>
+<label x="-22.86" y="127" size="1.27" layer="95" font="vector" xref="yes"/>
 </segment>
 </net>
@@
 <label x="45.72" y="109.22" size="1.27" layer="95" xref="yes"/>
 </segment>
+<segment>
+<pinref part="OPEN_CLOSE_TOGGLE" gate="G$1" pin="1"/>
+<wire x1="-91.44" y1="104.14" x2="-86.36" y2="104.14" width="0.1524" layer="91"/>
+<label x="-86.36" y="104.14" size="1.27" layer="95" xref="yes"/>
+</segment>
 </net>
 <net name="DEWAR_DIFF_ENABLE" class="0">
@@
 </segment>
 </net>
+<net name="DEWAR_FAULT_TRIGGER" class="0">
+<segment>
+<pinref part="DEWAR_SWITCH" gate="G$1" pin="2"/>
+<wire x1="-91.44" y1="134.62" x2="-88.9" y2="134.62" width="0.1524" layer="91"/>
+<label x="-88.9" y="134.62" size="1.27" layer="95" xref="yes"/>
+</segment>
+<segment>
+<portref moduleinst="BUFFER_OD1" port="A1"/>
+<wire x1="0" y1="116.84" x2="-2.54" y2="116.84" width="0.1524" layer="91"/>
+<label x="-2.54" y="116.84" size="1.27" layer="95" rot="R180" xref="yes"/>
+</segment>
+</net>
+<net name="SHUTTER_FAULT_TRIGGER" class="0">
+<segment>
+<pinref part="SHUTTER_SWITCH" gate="G$1" pin="2"/>
+<wire x1="-91.44" y1="121.92" x2="-88.9" y2="121.92" width="0.1524" layer="91"/>
+<label x="-88.9" y="121.92" size="1.27" layer="95" xref="yes"/>
+</segment>
+<segment>
+<portref moduleinst="BUFFER_OD1" port="A2"/>
+<wire x1="0" y1="111.76" x2="-2.54" y2="111.76" width="0.1524" layer="91"/>
+<label x="-2.54" y="111.76" size="1.27" layer="95" rot="R180" xref="yes"/>
+</segment>
+</net>
